File: Solder_Reflow_Oven_2.0.kicad_pcb (KiCad board)
At the start: 2 copper layers, 64.8 x 61.2 mm, 46 parts, among them J1 Conn_01x02_Male, J2 USB_B, J3 Conn_01x02_Male, J4 Conn_02x03_Top_Bottom, J5 Conn_01x02_Top_Bottom, J6 Conn_01x02_Male, J7 Conn_01x24_Male, Q1 2SD1805, SW1 SW_DIP_x01, U1 LM2940IMPX-10/NOPB, U2 MAX31855KASA, U3 RCLAMP0502A.TCT, U4 STM32L053R6T6, U5 CDBHD140L-G, U6 F24-100-C2, U7 SPDT_Reflow, Y1 Crystal_GND24

Commit message: Updating board for version 2.0.0
Parts:
- removed R10: R, Resistor_SMD:R_0805_2012Metric_Pad1.20x1.40mm_HandSolder
- removed R5: 1k, Resistor_SMD:R_0805_2012Metric_Pad1.20x1.40mm_HandSolder
- added U8: LD1117S33TR_SOT223, Package_TO_SOT_SMD:SOT-223-3_TabPin2, F.Cu at (99.5, 105.9)
- R4: value 2k -> 10
- moved R4 50.8 mm to (49.4, 121.8), turned to 270 degrees
- moved D1 1.86 mm to (91.1, 103.6), turned to 270 degrees
- moved R7 1.01 mm to (88.6, 103.6), turned to 90 degrees
- moved C10 0.91 mm to (94.7, 85.1)
- moved J2 0.09 mm to (46.5, 116.4)
- moved C13 0.06 mm to (96.5, 100.8)
- moved U1 0.05 mm to (99.0, 95.8)
Connections:
- R4 pad 1: VDD_10 -> VSS
- R4 pad 2: VDD_3.3 -> Net-(J2-Pad5)
- U6 pad 6: Net-(U6-Pad6) -> Net-(U5-Pad4)
- U6 pad 7: Net-(U6-Pad6) -> Net-(U6-Pad7)
- U6 pad 8: Net-(U5-Pad4) -> Net-(U6-Pad8)
Routing:
- net Net-(U5-Pad4): track 28.5 -> 11.9 mm
- net Net-(U6-Pad6): track 6.35 -> 0.00 mm
- net VDD_3.3: track 37.8 -> 33.7 mm
- net VDD_10: track 30.1 -> 33.7 mm
- net VSS: track 103.7 -> 101.4 mm, vias 36 -> 35
- net Net-(C10-Pad1): track 19.7 -> 18.7 mm
- net Net-(D1-Pad1): track 1.98 -> 2.50 mm
